File: TivaCtrlBoard.kicad_sch (KiCad schematic)
At the start: 96 parts

Commit message: Minor update
Parts:
- C1, C7: value (none) -> 2u2; footprint (none) -> Capacitor_SMD:C_0603_1608Metric_Pad1.08x0.95mm_HandSolder
- C10, C11, C15, C21, C22, C3, C5, C8, C9: value (none) -> 100n; footprint (none) -> Capacitor_SMD:C_0603_1608Metric_Pad1.08x0.95mm_HandSolder
- C12, C6: value (none) -> 1u; footprint (none) -> Capacitor_SMD:C_0603_1608Metric_Pad1.08x0.95mm_HandSolder
- C13, C14, C19, C2, C20, C4: value (none) -> 22p; footprint (none) -> Capacitor_SMD:C_0603_1608Metric_Pad1.08x0.95mm_HandSolder
- C16: value (none) -> 10n; footprint (none) -> Capacitor_SMD:C_0603_1608Metric_Pad1.08x0.95mm_HandSolder
- C17: value (none) -> 100n/30V; footprint (none) -> Capacitor_SMD:C_1206_3216Metric_Pad1.33x1.80mm_HandSolder
- C18: value (none) -> 10u/30V; footprint (none) -> Capacitor_SMD:C_1206_3216Metric_Pad1.33x1.80mm_HandSolder
- C23: value (none) -> 100p; footprint (none) -> Capacitor_SMD:C_0603_1608Metric_Pad1.08x0.95mm_HandSolder
- C24, C25, C26, C27: value (none) -> 10u; footprint (none) -> Capacitor_SMD:C_0805_2012Metric_Pad1.18x1.45mm_HandSolder
- D1: value (none) -> LED_BRG; footprint (none) -> LED_SMD:LED_RGB_5050-6
- D2, D3: value (none) -> D_Schottky; footprint (none) -> Diode_SMD:D_SMA_Handsoldering
- D4, D5, D6, D7, D8, D9: value (none) -> LED; footprint (none) -> sound_card_ctl:LED_0603_90rotated
- H1, H2, H3, H4: value (none) -> MountingHole; footprint (none) -> MountingHole:MountingHole_3.2mm_M3_DIN965_Pad_TopBottom
- IC1: value (none) -> LPH7366; footprint (none) -> sound_card_ctl:LPH7366
- J1: value (none) -> Screw_Terminal_01x02; footprint (none) -> TerminalBlock:TerminalBlock_bornier-2_P5.08mm
- J2: value (none) -> Conn_02x03_Odd_Even; footprint (none) -> Connector_PinHeader_2.54mm:PinHeader_2x03_P2.54mm_Vertical_SMD
- J3: value (none) -> Conn_01x04; footprint (none) -> Connector_PinHeader_2.54mm:PinHeader_1x05_P2.54mm_Vertical
- J4: value (none) -> Conn_02x10_Odd_Even; footprint (none) -> Connector_PinHeader_2.54mm:PinHeader_2x12_P2.54mm_Vertical_SMD
- J5: value (none) -> Conn_01x04; footprint (none) -> Connector_PinHeader_2.54mm:PinHeader_1x04_P2.54mm_Vertical
- L1, L3: value (none) -> 10u; footprint (none) -> Inductor_SMD:L_0603_1608Metric_Pad1.05x0.95mm_HandSolder
- L2: value (none) -> 10u; footprint (none) -> Inductor_SMD:L_Taiyo-Yuden_NR-60xx_HandSoldering
- Q1, Q2, Q3, Q4: value (none) -> BSN20; footprint (none) -> Package_TO_SOT_SMD:SOT-23
- R1, R4, R6: value (none) -> 330; footprint (none) -> Resistor_SMD:R_0603_1608Metric_Pad0.98x0.95mm_HandSolder
- R10, R18, R19, R25, R34, R7, R9: value (none) -> 100k; footprint (none) -> Resistor_SMD:R_0603_1608Metric_Pad0.98x0.95mm_HandSolder
- R11, R12, R20, R21: value (none) -> 4k7; footprint (none) -> Resistor_SMD:R_0603_1608Metric_Pad0.98x0.95mm_HandSolder
- R13, R14, R29, R3, R30: value (none) -> 10k; footprint (none) -> Resistor_SMD:R_0603_1608Metric_Pad0.98x0.95mm_HandSolder
- R15: value (none) -> R; footprint (none) -> Resistor_SMD:R_0603_1608Metric_Pad0.98x0.95mm_HandSolder
- R16, R17, R22, R23, R24, R26, R27, R28: value (none) -> 220; footprint (none) -> Resistor_SMD:R_0603_1608Metric_Pad0.98x0.95mm_HandSolder
- R2, R5, R8: value (none) -> 1k; footprint (none) -> Resistor_SMD:R_0603_1608Metric_Pad0.98x0.95mm_HandSolder
- R31, R32: value (none) -> 1M; footprint (none) -> Resistor_SMD:R_0603_1608Metric_Pad0.98x0.95mm_HandSolder
- R33: value (none) -> 22k; footprint (none) -> Resistor_SMD:R_0603_1608Metric_Pad0.98x0.95mm_HandSolder
- R35: value (none) -> 47; footprint (none) -> Resistor_SMD:R_0603_1608Metric_Pad0.98x0.95mm_HandSolder
- SW1, SW2: value (none) -> SW_SPST; footprint (none) -> sound_card_ctl:BTN_9mm_pitch5x5mm
- SW3: value (none) -> Rotary_Encoder_Switch; footprint (none) -> Rotary_Encoder:RotaryEncoder_Alps_EC12E-Switch_Vertical_H20mm_CircularMountingHoles
- U1: value (none) -> TM4C123GH6PM; footprint (none) -> Package_QFP:LQFP-64_10x10mm_P0.5mm
- U3: value (none) -> SRV05-4; footprint (none) -> Package_TO_SOT_SMD:SOT-23-6
- U4: value (none) -> TPS54202DDC; footprint (none) -> Package_TO_SOT_SMD:SOT-23-6
- Y1: value (none) -> 16MHz; footprint (none) -> Crystal:Crystal_SMD_5032-2Pin_5.0x3.2mm_HandSoldering
- Y2: value (none) -> 32.768k; footprint (none) -> Crystal:Crystal_C26-LF_D2.1mm_L6.5mm_Horizontal_1EP_style2
Other:
- title: (none) -> Tiva Control Board
